File: Apple/Apple IIc (PAL) - 050-0093-A/CPU_MMU_IOU_RAM.kicad_sch (KiCad schematic)
At the start: 24 parts

Commit message: starting to build a real iic
Parts:
- UD?: renamed from UD16; value 6502A -> 65c02; footprint (none) -> Package_DIP:DIP-40_W15.24mm; symbol Apple IIc Schematic Symbols:65C02A -> 65xx-library:W65C02SxP
- UD?: renamed from UD4; footprint (none) -> Package_DIP:DIP-20_W7.62mm_Socket
- UD?: renamed from UD18; value 27256 -> 27c256
- UE?: renamed from UE16; footprint (none) -> Package_DIP:DIP-40_W15.24mm
- UE?: renamed from UE14; footprint (none) -> Package_DIP:DIP-40_W15.24mm
- UF?: renamed from UF19; value 6664 -> MK4164N; footprint (none) -> Package_DIP:DIP-16_W7.62mm; symbol Apple IIc Schematic Symbols:6664 -> Memory_RAM:MK4164N
- UF?: renamed from UF17; value 6664 -> MK4164N; footprint (none) -> Package_DIP:DIP-16_W7.62mm; symbol Apple IIc Schematic Symbols:6664 -> Memory_RAM:MK4164N
- UF?: renamed from UF12; value 6664 -> MK4164N; footprint (none) -> Package_DIP:DIP-16_W7.62mm; symbol Apple IIc Schematic Symbols:6664 -> Memory_RAM:MK4164N
- UF?: renamed from UF16; value 6664 -> MK4164N; footprint (none) -> Package_DIP:DIP-16_W7.62mm; symbol Apple IIc Schematic Symbols:6664 -> Memory_RAM:MK4164N
- UF?: renamed from UF14; value 6664 -> MK4164N; footprint (none) -> Package_DIP:DIP-16_W7.62mm; symbol Apple IIc Schematic Symbols:6664 -> Memory_RAM:MK4164N
- UF?: renamed from UF13; value 6664 -> MK4164N; footprint (none) -> Package_DIP:DIP-16_W7.62mm; symbol Apple IIc Schematic Symbols:6664 -> Memory_RAM:MK4164N
- UF?: renamed from UF18; value 6664 -> MK4164N; footprint (none) -> Package_DIP:DIP-16_W7.62mm; symbol Apple IIc Schematic Symbols:6664 -> Memory_RAM:MK4164N
- UF?: renamed from UF15; value 6664 -> MK4164N; footprint (none) -> Package_DIP:DIP-16_W7.62mm; symbol Apple IIc Schematic Symbols:6664 -> Memory_RAM:MK4164N
- renumbered CR3 to CR?, CR2 to CR?, R1 to R?, R2 to R?, RP5 to RP3, RP11 to RP?, RP1 to RP?, W2 to W?, W1 to W?
Connections:
- net +5V: now also RP?.1 (R1.1); no longer UF?.1 (~{REFRESH}), UF?.1 (~{REFRESH}), UF?.1 (~{REFRESH}), UF?.1 (~{REFRESH}), UF?.1 (~{REFRESH}), UF?.1 (~{REFRESH}), UF?.1 (~{REFRESH}), UF?.1 (~{REFRESH})
- net RA1: now also UF?.7 (A1), UF?.7 (A1), UF?.7 (A1), UF?.7 (A1), UF?.7 (A1), UF?.7 (A1), UF?.7 (A1), UF?.7 (A1); no longer UF?.6, UF?.6, UF?.6, UF?.6, UF?.6, UF?.6, UF?.6, UF?.6
- net RA2: now also UF?.6 (A2), UF?.6 (A2), UF?.6 (A2), UF?.6 (A2), UF?.6 (A2), UF?.6 (A2), UF?.6 (A2), UF?.6 (A2); no longer UF?.7, UF?.7, UF?.7, UF?.7, UF?.7, UF?.7, UF?.7, UF?.7
- net RA3: now also UF?.12 (A3), UF?.12 (A3), UF?.12 (A3), UF?.12 (A3), UF?.12 (A3), UF?.12 (A3), UF?.12 (A3), UF?.12 (A3); no longer UF?.10, UF?.10, UF?.10, UF?.10, UF?.10, UF?.10, UF?.10, UF?.10
- net RA5: now also UF?.10 (A5), UF?.10 (A5), UF?.10 (A5), UF?.10 (A5), UF?.10 (A5), UF?.10 (A5), UF?.10 (A5), UF?.10 (A5); no longer UF?.12, UF?.12, UF?.12, UF?.12, UF?.12, UF?.12, UF?.12, UF?.12
- net S5: now also RP?.2 (R1.2); no longer RP?.4 (R3.2)
- net ~{IRQ}: now also RP1.2 (R1.2); no longer RP1.4 (R3.2)
- net ~{RAS}: no longer R?.2
- net ~{ROMEN}: now also RP1.2 (R1.2); no longer RP1.4 (R3.2)
- net ~{ROMOE}: now also RP3.2 (R1.2); no longer RP3.3 (R2.2)
- net at UD?.11 (~{TMGEN}): now also RP?.2 (R1.2); no longer RP?.5 (R4.2)
- no-connect marks 1 -> 0
Other:
- moved on the sheet: R?
