File: Apple/Apple IIc (PAL) - 050-0093-A/IWM.kicad_sch (KiCad schematic)
At the start: 3 parts, among them J2 External Disk, J8 Internal Disk

Commit message: starting to build a real iic
Parts:
- J?: renamed from J8; footprint (none) -> Connector_IDC:IDC-Header_2x10_P2.54mm_Vertical
- UD?: renamed from UD2; footprint (none) -> Package_DIP:DIP-28_W15.24mm
- renumbered J2 to J?
