File: Apple/Apple IIc (PAL) - 050-0093-A/Power.kicad_sch (KiCad schematic)
At the start: 56 parts, among them J1 External Power In, J11 Power Supply

Commit message: starting to build a real iic
Parts:
- renumbered C59 to C48, C57 to C49, C60 to C50, UB13 to UB2
Changed lines of the file:
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@@
 (kicad_sch
-	(version 20231120)
+	(version 20250114)
 	(generator "eeschema")
-	(generator_version "8.0")
+	(generator_version "9.0")
 	(paper "A4")
 	(title_block
@@
 		(comment 1 "Apple IIc ROM255")
 	)
+	(text "ON"
+		(exclude_from_sim no)
+		(at 245.745 127.635 0)
+		(effects
+			(font
+				(size 1.27 1.27)
+			)
+			(justify left bottom)
+		)
+	)
+	(text "No value given for C1-C64"
+		(exclude_from_sim no)
+		(at 80.01 61.595 0)
+		(effects
+			(font
+				(face "Verdana")
+				(size 1.27 1.27)
+				(color 0 0 194 1)
+			)
+			(justify left bottom)
+		)
+	)
+	(text "OFF"
+		(exclude_from_sim no)
+		(at 258.445 127 0)
+		(effects
+			(font
+				(size 1.27 1.27)
+			)
+			(justify left bottom)
+		)
+	)
+	(text "TODO: Is this right? \nOFF is wired to +12VIN?"
+		(exclude_from_sim no)
+		(at 242.57 139.7 0)
+		(effects
+			(font
+				(face "Verdana")
+				(size 1.27 1.27)
+			)
+			(justify left bottom)
+		)
+	)
+	(text "TODO: Look at C60 on real IIc"
+		(exclude_from_sim no)
+		(at 198.755 93.98 0)
+		(effects
+			(font
+				(face "Verdana")
+				(size 1.27 1.27)
+			)
+			(justify left bottom)
+		)
+	)
+	(text "Verify: No C52 in OG schematic?"
+		(exclude_from_sim no)
+		(at 15.875 56.515 0)
+		(effects
+			(font
+				(face "Verdana")
+				(size 1.27 1.27)
+				(color 0 0 194 1)
+			)
+			(justify left bottom)
+		)
+	)
 	(junction
 		(at 140.335 116.205)
@@
 		)
 	)
-	(text "ON"
-		(exclude_from_sim no)
-		(at 245.745 127.635 0)
-		(effects
-			(font
-				(size 1.27 1.27)
-			)
-			(justify left bottom)
-		)
-	)
-	(text "No value given for C1-C64"
-		(exclude_from_sim no)
-		(at 80.01 61.595 0)
-		(effects
-			(font
-				(face "Verdana")
-				(size 1.27 1.27)
-				(color 0 0 194 1)
-			)
-			(justify left bottom)
-		)
-	)
-	(text "OFF"
-		(exclude_from_sim no)
-		(at 258.445 127 0)
-		(effects
-			(font
-				(size 1.27 1.27)
-			)
-			(justify left bottom)
-		)
-	)
-	(text "TODO: Is this right? \nOFF is wired to +12VIN?"
-		(exclude_from_sim no)
-		(at 242.57 139.7 0)
-		(effects
-			(font
-				(face "Verdana")
-				(size 1.27 1.27)
-			)
-			(justify left bottom)
-		)
-	)
-	(text "TODO: Look at C60 on real IIc"
-		(exclude_from_sim no)
-		(at 198.755 93.98 0)
-		(effects
-			(font
-				(face "Verdana")
-				(size 1.27 1.27)
-			)
-			(justify left bottom)
-		)
-	)
-	(text "Verify: No C52 in OG schematic?"
-		(exclude_from_sim no)
-		(at 15.875 56.515 0)
-		(effects
-			(font
-				(face "Verdana")
-				(size 1.27 1.27)
-				(color 0 0 194 1)
-			)
-			(justify left bottom)
-		)
-	)
 	(label "EEE"
 		(at 168.91 137.795 0)
-		(fields_autoplaced yes)
 		(effects
 			(font
@@
 	(label "GND"
 		(at 142.24 128.905 180)
-		(fields_autoplaced yes)
 		(effects
 			(font
@@
 	(label "DDD"
 		(at 168.91 119.38 0)
-		(fields_autoplaced yes)
 		(effects
 			(font
@@
 	(label "AAA"
 		(at 118.745 180.975 0)
-		(fields_autoplaced yes)
 		(effects
 			(font
@@
 	(label "FFF"
 		(at 252.73 118.11 0)
-		(fields_autoplaced yes)
 		(effects
 			(font
@@
 	(label "BBB"
 		(at 144.145 180.975 180)
-		(fields_autoplaced yes)
 		(effects
 			(font
@@
 	(label "EEE"
 		(at 144.145 175.895 180)
-		(fields_autoplaced yes)
 		(effects
 			(font
@@
 	(label "GND"
 		(at 142.24 100.965 180)
-		(fields_autoplaced yes)
 		(effects
 			(font
@@
 	(label "CCC"
 		(at 118.745 175.895 0)
-		(fields_autoplaced yes)
 		(effects
 			(font
@@
 	(label "GND"
 		(at 142.24 131.445 180)
-		(fields_autoplaced yes)
 		(effects
 			(font
@@
 	(label "CCC"
 		(at 168.91 116.205 0)
-		(fields_autoplaced yes)
 		(effects
 			(font
@@
 	(label "FFF"
 		(at 168.91 113.665 0)
-		(fields_autoplaced yes)
 		(effects
 			(font
@@
 	(label "DDD"
 		(at 139.065 168.91 180)
-		(fields_autoplaced yes)
 		(effects
 			(font
@@
 	(label "FFF"
 		(at 140.335 113.665 0)
-		(fields_autoplaced yes)
 		(effects
 			(font
@@
 	(label "GND"
 		(at 142.24 151.765 180)
-		(fields_autoplaced yes)
 		(effects
 			(font
@@
 	(label "GND"
 		(at 142.24 154.305 180)
-		(fields_autoplaced yes)
 		(effects
 			(font
@@
 	(label "GND"
 		(at 142.24 103.505 180)
-		(fields_autoplaced yes)
 		(effects
 			(font
@@
 		(shape output)
 		(at 118.11 180.975 180)
-		(fields_autoplaced yes)
 		(effects
 			(font
@@
 		(shape output)
 		(at 150.495 116.205 0)
-		(fields_autoplaced yes)
 		(effects
 			(font
@@
 		(shape output)
 		(at 144.78 180.975 0)
-		(fields_autoplaced yes)
 		(effects
 			(font
@@
 		(dnp no)
 		(fields_autoplaced yes)
-		(property "Reference" "#PWR049"
+		(property "Reference" "#PWR048"
 			(at 203.835 92.075 0)
 			(effects
@@
 		(dnp no)
 		(fields_autoplaced yes)
-		(property "Reference" "C59"
+		(property "Reference" "C48"
 			(at 192.405 127.6413 0)
 			(effects
@@
 		(dnp no)
 		(fields_autoplaced yes)
-		(property "Reference" "#PWR048"
+		(property "Reference" "#PWR050"
 			(at 219.075 80.645 0)
 			(effects
@@
 		(dnp no)
 		(fields_autoplaced yes)
-		(property "Reference" "#PWR043"
+		(property "Reference" "#PWR040"
 			(at 189.23 139.7 0)
 			(effects
@@
 		(dnp no)
 		(fields_autoplaced yes)
-		(property "Reference" "#PWR040"
+		(property "Reference" "#PWR043"
 			(at 235.585 132.08 0)
 			(effects
@@
 		(on_board yes)
 		(dnp no)
-		(property "Reference" "#PWR044"
+		(property "Reference" "#PWR045"
 			(at 271.78 127.635 0)
 			(effects
@@
 		(on_board yes)
 		(dnp no)
-		(property "Reference" "C60"
+		(property "Reference" "C50"
 			(at 210.185 78.74 0)
 			(effects
@@
 		(dnp no)
 		(fields_autoplaced yes)
-		(property "Reference" "#PWR042"
+		(property "Reference" "#PWR039"
 			(at 175.895 139.7 0)
 			(effects
@@
 		(dnp no)
 		(fields_autoplaced yes)
-		(property "Reference" "#FLG01"
+		(property "Reference" "#FLG02"
 			(at 231.14 120.65 0)
 			(effects
@@
 		(dnp no)
 		(fields_autoplaced yes)
-		(property "Reference" "#FLG02"
+		(property "Reference" "#FLG01"
 			(at 231.775 127.635 0)
 			(effects
@@
 		(dnp no)
 		(fields_autoplaced yes)
-		(property "Reference" "#PWR045"
+		(property "Reference" "#PWR044"
 			(at 250.19 135.89 0)
 			(effects
@@
 		(dnp no)
 		(fields_autoplaced yes)
-		(property "Reference" "#PWR050"
+		(property "Reference" "#PWR049"
 			(at 215.265 90.17 0)
 			(effects
@@
 		(on_board yes)
 		(dnp no)
-		(property "Reference" "C57"
+		(property "Reference" "C49"
 			(at 274.32 130.175 0)
 			(effects
@@
 		(dnp no)
 		(fields_autoplaced yes)
-		(property "Reference" "#PWR039"
+		(property "Reference" "#PWR042"
 			(at 234.315 123.825 0)
 			(effects
@@
 		(on_board yes)
 		(dnp no)
-		(property "Reference" "UB13"
+		(property "Reference" "UB2"
 			(at 203.835 71.12 0)
 			(effects
