File: Apple/Apple IIc (PAL) - 050-0093-A/Serial and GLU.kicad_sch (KiCad schematic)
At the start: 35 parts, among them J12 Serial 2, J6 Serial 1, Q1 2n2369, X1 OSC, Y1 1.8432 MHz

Commit message: starting to build a real iic
Parts:
- UB18, UC18: footprint (none) -> Package_DIP:DIP-8_W7.62mm
- UC11, UC4, UC9: footprint (none) -> Package_DIP:DIP-14_W7.62mm
- UC7: footprint (none) -> Package_DIP:DIP-16_W7.62mm
- UD11, UD9: footprint (none) -> Package_DIP:DIP-28_W15.24mm
- UD6: footprint (none) -> Package_DIP:DIP-24_18.0mmx34.29mm_W15.24mm
- X1: footprint (none) -> Oscillator:Oscillator_DIP-14
Connections:
- net +5V: no longer UC9.14 (VCC)
- net DSR2B: now also UC4.5 (nc)
- net GND: no longer UC9.7 (GND)
- net PH1: now also UC9.1; no longer UC9.4
- net RD1B: now also UC4.12 (nc)
- net RR/~{W}: now also UC9.3; no longer UC9.6
- net R/~{W}: now also UC9.2; no longer UC9.5
- net ~{GLUEN}: now also RP11.2 (R1.2); no longer RP11.5 (R4.2)
- net ~{IOUSELIO}: now also UC9.3; no longer UC9.8
- net ~{SELIO}: now also UC9.1; no longer UC9.9
- net at C51.1, R15.2, UC18.2 (TR)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: now also UC18.5 (nc)
- net at Q1.3 (C), R20.2: now also UC9.2; no longer UC9.10
