File: Apple/Apple IIc (PAL) - 050-0093-A/Video.kicad_sch (KiCad schematic)
At the start: 22 parts, among them J4 Video, J5 Video, U1 VID

Commit message: starting to build a real iic
Parts:
- UF10, UF11, UF4, UF5, UF6, UF7, UF8, UF9: value 6664 -> MK4164N; footprint (none) -> Package_DIP:DIP-16_W7.62mm; symbol Apple IIc Schematic Symbols:6664 -> Memory_RAM:MK4164N
Connections:
- net +5V: no longer UF10.1 (~{REFRESH}), UF10.8 (VCC), UF11.1 (~{REFRESH}), UF11.8 (VCC), UF4.1 (~{REFRESH}), UF4.8 (VCC), UF5.1 (~{REFRESH}), UF5.8 (VCC), UF6.1 (~{REFRESH}), UF6.8 (VCC), UF7.1 (~{REFRESH}), UF7.8 (VCC), UF8.1 (~{REFRESH}), UF8.8 (VCC), UF9.1 (~{REFRESH}), UF9.8 (VCC)
- net ALT0: no longer UF11.14 (Q), UF11.2 (D)
- net ALT1: no longer UF10.14 (Q), UF10.2 (D)
- net ALT2: no longer UF9.14 (Q), UF9.2 (D)
- net ALT3: no longer UF8.14 (Q), UF8.2 (D)
- net ALT4: no longer UF7.14 (Q), UF7.2 (D)
- net ALT5: no longer UF6.14 (Q), UF6.2 (D)
- net ALT6: no longer UF5.14 (Q), UF5.2 (D)
- net ALT7: no longer UF4.14 (Q), UF4.2 (D)
- net GND: no longer UF10.16 (VSS), UF11.16 (VSS), UF4.16 (VSS), UF5.16 (VSS), UF6.16 (VSS), UF7.16 (VSS), UF8.16 (VSS), UF9.16 (VSS)
- net Q3b: no longer UF10.15 (~{CAS}), UF11.15 (~{CAS}), UF4.15 (~{CAS}), UF5.15 (~{CAS}), UF6.15 (~{CAS}), UF7.15 (~{CAS}), UF8.15 (~{CAS}), UF9.15 (~{CAS})
- net RA0: no longer UF10.5, UF11.5, UF4.5, UF5.5, UF6.5, UF7.5, UF8.5, UF9.5
- net RA1: no longer UF10.6, UF11.6, UF4.6, UF5.6, UF6.6, UF7.6, UF8.6, UF9.6
- net RA2: no longer UF10.7, UF11.7, UF4.7, UF5.7, UF6.7, UF7.7, UF8.7, UF9.7
- net RA3: no longer UF10.10, UF11.10, UF4.10, UF5.10, UF6.10, UF7.10, UF8.10, UF9.10
- net RA4: no longer UF10.11, UF11.11, UF4.11, UF5.11, UF6.11, UF7.11, UF8.11, UF9.11
- net RA5: no longer UF10.12, UF11.12, UF4.12, UF5.12, UF6.12, UF7.12, UF8.12, UF9.12
- net RA6: no longer UF10.13, UF11.13, UF4.13, UF5.13, UF6.13, UF7.13, UF8.13, UF9.13
- net RA7: no longer UF10.9, UF11.9, UF4.9, UF5.9, UF6.9, UF7.9, UF8.9, UF9.9
- net R/~{W}80: no longer UF10.3 (~{W}), UF11.3 (~{W}), UF4.3 (~{W}), UF5.3 (~{W}), UF6.3 (~{W}), UF7.3 (~{W}), UF8.3 (~{W}), UF9.3 (~{W})
- net ~{PRASb}: no longer UF10.4 (~{RAS}), UF11.4 (~{RAS}), UF4.4 (~{RAS}), UF5.4 (~{RAS}), UF6.4 (~{RAS}), UF7.4 (~{RAS}), UF8.4 (~{RAS}), UF9.4 (~{RAS})
