File: Apple/Apple IIc (PAL) - 050-0093-A/keyboard_and_gameport.kicad_sch (KiCad schematic)
At the start: 23 parts, among them J3 Game, J9 Keyboard

Commit message: starting to build a real iic
Parts:
- J?: renamed from J3; footprint (none) -> Connector_Dsub:DSUB-9_Pins_Horizontal_P2.77x2.54mm_EdgePinOffset9.40mm
- J?: renamed from J9; footprint (none) -> Connector_IDC:IDC-Header_2x17_P2.54mm_Vertical
- RP4: footprint (none) -> Connector_PinSocket_2.54mm:PinSocket_1x06_P2.54mm_Vertical
- UB?: renamed from UB16; footprint (none) -> Package_DIP:DIP-40_W15.24mm
- UD?: renamed from UD16; footprint (none) -> Package_DIP:DIP-22_W10.16mm
- UF?: renamed from UF1; footprint (none) -> Package_DIP:DIP-16_W7.62mm
- UF?: renamed from UF2; footprint (none) -> Package_DIP:DIP-14_W7.62mm
- UF?: renamed from UF3; footprint (none) -> Package_DIP:DIP-16_W7.62mm
- renumbered C45 to C?, C49 to C?, C46 to C?, C47 to C?, R18 to R?, R7 to R?, R6 to R?, R8 to R?, RP10 to RP?, RP1 to RP?, RP9 to RP?, RP11 to RP?
Connections:
- net CAPS: now also RP?.2 (R1.2); no longer RP?.5 (R4.2)
- net CONTROL: now also RP?.2 (R1.2); no longer RP?.7 (R6.2)
- net CP0: now also RP?.2 (R1.2); no longer RP?.4 (R3.2)
- net CP1: now also RP?.2 (R1.2); no longer RP?.4 (R3.2)
- net LANGSW: now also RP?.2 (R1.2); no longer RP?.5 (R4.2)
- net SHIFT: now also RP?.2 (R1.2); no longer RP?.6 (R5.2)
- net ~{RESET}: now also RP?.2 (R1.2); no longer RP?.4 (R3.2)
- new net: UB?.32 (nc), UB?.4 (nc)
