File: Apple/Apple IIc (PAL) - 050-0093-A/sound.kicad_sch (KiCad schematic)
At the start: 9 parts, among them J10 Internal Speaker, J7 Earphone

Commit message: starting to build a real iic
Parts:
- renumbered C44 to C31, C43 to C32, L6 to L5, L5 to L6, UA14 to UA1
Changed lines of the file:
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@@
 (kicad_sch
-	(version 20231120)
+	(version 20250114)
 	(generator "eeschema")
-	(generator_version "8.0")
+	(generator_version "9.0")
 	(paper "A3")
 	(title_block
@@
 	(label "EAROUT"
 		(at 306.705 122.555 180)
-		(fields_autoplaced yes)
 		(effects
 			(font
@@
 	(label "EAROUT2"
 		(at 306.705 120.015 180)
-		(fields_autoplaced yes)
 		(effects
 			(font
@@
 	(label "EARGND"
 		(at 280.035 123.19 0)
-		(fields_autoplaced yes)
 		(effects
 			(font
@@
 	(label "EAROUT1"
 		(at 306.705 127.635 180)
-		(fields_autoplaced yes)
 		(effects
 			(font
@@
 	(label "EAROUT1"
 		(at 311.785 104.775 180)
-		(fields_autoplaced yes)
 		(effects
 			(font
@@
 	(label "EAROUT2"
 		(at 311.785 107.315 180)
-		(fields_autoplaced yes)
 		(effects
 			(font
@@
 		(shape output)
 		(at 305.435 94.615 0)
-		(fields_autoplaced yes)
 		(effects
 			(font
@@
 		(shape input)
 		(at 198.755 90.805 180)
-		(fields_autoplaced yes)
 		(effects
 			(font
@@
 		(dnp no)
 		(fields_autoplaced yes)
-		(property "Reference" "#PWR0108"
+		(property "Reference" "#PWR0106"
 			(at 234.315 110.49 0)
 			(effects
@@
 		(on_board yes)
 		(dnp no)
-		(property "Reference" "C44"
+		(property "Reference" "C31"
 			(at 250.825 102.235 0)
 			(effects
@@
 		(dnp no)
 		(fields_autoplaced yes)
-		(property "Reference" "#PWR0109"
+		(property "Reference" "#PWR0152"
 			(at 320.675 133.985 0)
 			(effects
@@
 		(on_board yes)
 		(dnp no)
-		(property "Reference" "L6"
+		(property "Reference" "L5"
 			(at 277.495 102.87 90)
 			(effects
@@
 		(dnp no)
 		(fields_autoplaced yes)
-		(property "Reference" "#PWR0107"
+		(property "Reference" "#PWR0108"
 			(at 248.285 93.98 0)
 			(effects
@@
 		(dnp no)
 		(fields_autoplaced yes)
-		(property "Reference" "#PWR0105"
+		(property "Reference" "#PWR0107"
 			(at 248.285 81.915 0)
 			(effects
@@
 		(on_board yes)
 		(dnp no)
-		(property "Reference" "UA14"
+		(property "Reference" "UA1"
 			(at 231.775 87.63 0)
 			(effects
@@
 		(on_board yes)
 		(dnp no)
-		(property "Reference" "L5"
+		(property "Reference" "L6"
 			(at 276.86 124.46 90)
 			(effects
@@
 		(dnp no)
 		(fields_autoplaced yes)
-		(property "Reference" "#PWR0106"
+		(property "Reference" "#PWR0105"
 			(at 234.315 80.645 0)
 			(effects
@@
 		(on_board yes)
 		(dnp no)
-		(property "Reference" "C43"
+		(property "Reference" "C32"
 			(at 262.89 99.695 0)
 			(effects
